File: snes_maskrom_psop_to_dip_adapter/snes_maskrom_psop_to_dip_adapter.kicad_pcb (KiCad board)
At the start: 2 copper layers, 20.4 x 46.4 mm, 5 parts, among them U1 MASKROM, U3 29F1610

Commit message: update img and gerbers
Parts:
- added JP2: WE`, Jumper:SolderJumper-2_P1.3mm_Open_RoundedPad1.0x1.5mm, B.Cu at (124.3, 71.3)
- JP1: value WE`/WP` -> WP`; footprint Jumper:SolderJumper-3_P1.3mm_Open_RoundedPad1.0x1.5mm_NumberLabels -> Jumper:SolderJumper-2_P1.3mm_Open_RoundedPad1.0x1.5mm
- moved JP1 0.60 mm to (120.9, 71.3)
Routing:
- net /Vcc: track 46.3 -> 48.9 mm, vias 1 -> 2
- net /WE`: track 11.0 -> 8.98 mm
Other:
- board text added: "snes psop2maskrom rev2 papkor 05.26 vk.com/games_hw"
- board text removed: "snes psop2maskrom papkor 06.25"
