File: snes_maskrom_psop_to_dip_adapter/snes_maskrom_psop_to_dip_adapter.kicad_sch (KiCad schematic)
At the start: 5 parts, among them U1 MASKROM, U3 29F1610

Commit message: update img and gerbers
Parts:
- added JP2: WE`, Jumper:SolderJumper-2_P1.3mm_Open_RoundedPad1.0x1.5mm, symbol Jumper:SolderJumper_2_Open
- JP1: value WE`/WP` -> WP`; footprint Jumper:SolderJumper-3_P1.3mm_Open_RoundedPad1.0x1.5mm_NumberLabels -> Jumper:SolderJumper-2_P1.3mm_Open_RoundedPad1.0x1.5mm; symbol Jumper:SolderJumper_3_Open -> Jumper:SolderJumper_2_Open
Connections:
- net Vcc: now also JP2.1 (A)
- net WE`: now also JP2.2 (B); no longer JP1.3 (B)
Changed lines of the file:
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@@
 	(generator_version "9.0")
 	(paper "A4")
+	(title_block
+		(rev "2")
+	)
 	(junction
 		(at 130.81 48.26)
@@
 	)
 	(bus_entry
-		(at 128.27 59.69)
+		(at 128.27 52.07)
 		(size 2.54 -2.54)
 		(stroke
@@
 	)
 	(bus_entry
+		(at 128.27 59.69)
+		(size 2.54 -2.54)
+		(stroke
+			(width 0)
+			(type default)
+		)
+	)
+	(bus_entry
 		(at 66.04 80.01)
 		(size 2.54 2.54)
@@
 	)
 	(bus_entry
-		(at 128.27 69.85)
+		(at 128.27 73.66)
 		(size 2.54 -2.54)
 		(stroke
@@
 	)
 	(bus_entry
-		(at 128.27 64.77)
+		(at 128.27 66.04)
 		(size 2.54 -2.54)
 		(stroke
@@
 		)
 	)
+	(wire
+		(pts
+			(xy 118.11 66.04) (xy 128.27 66.04)
+		)
+		(stroke
+			(width 0)
+			(type default)
+		)
+	)
 	(bus
 		(pts
@@
 	(wire
 		(pts
-			(xy 118.11 69.85) (xy 128.27 69.85)
+			(xy 118.11 73.66) (xy 128.27 73.66)
 		)
 		(stroke
@@
 		)
 	)
+	(bus
+		(pts
+			(xy 130.81 59.69) (xy 130.81 62.23)
+		)
+		(stroke
+			(width 0)
+			(type default)
+		)
+	)
 	(wire
 		(pts
@@
 	(bus
 		(pts
-			(xy 130.81 62.23) (xy 130.81 64.77)
+			(xy 130.81 62.23) (xy 130.81 63.5)
 		)
 		(stroke
@@
 		)
 	)
+	(bus
+		(pts
+			(xy 130.81 69.85) (xy 130.81 71.12)
+		)
+		(stroke
+			(width 0)
+			(type default)
+		)
+	)
 	(wire
 		(pts
-			(xy 118.11 59.69) (xy 128.27 59.69)
+			(xy 118.11 52.07) (xy 128.27 52.07)
 		)
 		(stroke
@@
 		)
 	)
+	(bus
+		(pts
+			(xy 130.81 63.5) (xy 130.81 64.77)
+		)
+		(stroke
+			(width 0)
+			(type default)
+		)
+	)
 	(wire
 		(pts
@@
 		)
 	)
-	(bus
+	(wire
 		(pts
-			(xy 130.81 69.85) (xy 130.81 72.39)
+			(xy 151.13 100.33) (xy 157.48 100.33)
 		)
 		(stroke
@@
 		)
 	)
-	(wire
+	(bus
 		(pts
-			(xy 151.13 100.33) (xy 157.48 100.33)
+			(xy 130.81 71.12) (xy 130.81 72.39)
 		)
 		(stroke
@@
 	(bus
 		(pts
-			(xy 130.81 48.26) (xy 130.81 57.15)
+			(xy 130.81 48.26) (xy 130.81 49.53)
 		)
 		(stroke
@@
 	(wire
 		(pts
-			(xy 133.35 90.17) (xy 138.43 90.17)
+			(xy 118.11 59.69) (xy 128.27 59.69)
 		)
 		(stroke
@@
 		)
 	)
-	(bus
+	(wire
 		(pts
-			(xy 130.81 102.87) (xy 130.81 107.95)
+			(xy 133.35 90.17) (xy 138.43 90.17)
 		)
 		(stroke
@@
 	(bus
 		(pts
-			(xy 93.98 74.93) (xy 93.98 77.47)
+			(xy 130.81 102.87) (xy 130.81 107.95)
 		)
 		(stroke
@@
 	(bus
 		(pts
-			(xy 130.81 64.77) (xy 130.81 67.31)
+			(xy 93.98 74.93) (xy 93.98 77.47)
 		)
 		(stroke
@@
 		)
 	)
+	(bus
+		(pts
+			(xy 130.81 64.77) (xy 130.81 67.31)
+		)
+		(stroke
+			(width 0)
+			(type default)
+		)
+	)
 	(wire
 		(pts
@@
 	(bus
 		(pts
-			(xy 130.81 59.69) (xy 130.81 62.23)
-		)
-		(stroke
-			(width 0)
-			(type default)
-		)
-	)
-	(bus
-		(pts
 			(xy 160.02 92.71) (xy 160.02 97.79)
 		)
@@
 		)
 	)
-	(wire
+	(bus
 		(pts
-			(xy 86.36 102.87) (xy 91.44 102.87)
+			(xy 130.81 49.53) (xy 130.81 57.15)
 		)
 		(stroke
@@
 	(wire
 		(pts
-			(xy 121.92 64.77) (xy 128.27 64.77)
+			(xy 86.36 102.87) (xy 91.44 102.87)
 		)
 		(stroke
@@
 	)
 	(label "Vss"
-		(at 123.19 64.77 0)
+		(at 123.19 66.04 0)
 		(effects
 			(font
@@
 		)
 	)
+	(label "Vcc"
+		(at 123.19 59.69 0)
+		(effects
+			(font
+				(size 1.27 1.27)
+			)
+			(justify left bottom)
+		)
+	)
 	(label "A16"
 		(at 152.4 82.55 0)
@@
 	)
 	(label "WE`"
-		(at 123.19 59.69 0)
+		(at 123.19 52.07 0)
 		(effects
 			(font
@@
 	)
 	(label "WP`"
-		(at 123.19 69.85 0)
+		(at 123.19 73.66 0)
 		(effects
 			(font
@@
 	)
 	(symbol
-		(lib_id "Jumper:SolderJumper_3_Open")
-		(at 118.11 64.77 90)
+		(lib_name "SolderJumper_2_Open_1")
+		(lib_id "Jumper:SolderJumper_2_Open")
+		(at 118.11 69.85 90)
 		(unit 1)
 		(exclude_from_sim no)
@@
 		(fields_autoplaced yes)
 		(property "Reference" "JP1"
-			(at 115.57 63.4999 90)
+			(at 120.65 68.5799 90)
 			(effects
 				(font
 					(size 1.27 1.27)
 				)
-				(justify left)
+				(justify right)
 			)
 		)
-		(property "Value" "WE`/WP`"
-			(at 115.57 66.0399 90)
+		(property "Value" "WP`"
+			(at 120.65 71.1199 90)
 			(effects
 				(font
 					(size 1.27 1.27)
 				)
-				(justify left)
+				(justify right)
 			)
 		)
-		(property "Footprint" "Jumper:SolderJumper-3_P1.3mm_Open_RoundedPad1.0x1.5mm_NumberLabels"
-			(at 118.11 64.77 0)
+		(property "Footprint" "Jumper:SolderJumper-2_P1.3mm_Open_RoundedPad1.0x1.5mm"
+			(at 118.11 69.85 0)
 			(effects
 				(font
@@
 		)
 		(property "Datasheet" "~"
-			(at 118.11 64.77 0)
+			(at 118.11 69.85 0)
 			(effects
 				(font
@@
 			)
 		)
-		(property "Description" "Solder Jumper, 3-pole, open"
-			(at 118.11 64.77 0)
+		(property "Description" "Solder Jumper, 2-pole, open"
+			(at 118.11 69.85 0)
 			(effects
 				(font
@@
 		(pin "1"
 		)
-		(pin "3"
-		)
 		(pin "2"
 		)
@@
 					(unit 1)
 				)
+			)
+		)
+	)
+	(symbol
+		(lib_id "Jumper:SolderJumper_2_Open")
+		(at 118.11 55.88 90)
+		(unit 1)
+		(exclude_from_sim no)
+		(in_bom no)
+		(on_board yes)
+		(dnp no)
+		(property "Reference" "JP2"
+			(at 112.014 54.61 90)
+			(effects
+				(font
+					(size 1.27 1.27)
+				)
+				(justify right)
+			)
+		)
+		(property "Value" "WE`"
+			(at 112.268 56.896 90)
+			(effects
+				(font
+					(size 1.27 1.27)
+				)
+				(justify right)
+			)
+		)
+		(property "Footprint" "Jumper:SolderJumper-2_P1.3mm_Open_RoundedPad1.0x1.5mm"
+			(at 118.11 55.88 0)
+			(effects
+				(font
+					(size 1.27 1.27)
+				)
+				(hide yes)
+			)
+		)
+		(property "Datasheet" "~"
+			(at 118.11 55.88 0)
+			(effects
+				(font
+					(size 1.27 1.27)
+				)
+				(hide yes)
+			)
+		)
+		(property "Description" "Solder Jumper, 2-pole, open"
+			(at 118.11 55.88 0)
+			(effects
+				(font
+					(size 1.27 1.27)
+				)
+				(hide yes)
+			)
+		)
+		(pin "1"
+		)
+		(pin "2"
+		)
+		(instances
+			(project "snes_maskrom_psop_to_dip_adapter"
+				(path "/04238f28-9b6b-499e-bfd3-7cbdeddf7961"
+					(reference "JP2")
+					(unit 1)
+				)
