File: snes_maskrom_tsop_to_dip_adapter/snes_maskrom_tsop_to_dip_adapter.kicad_pcb (KiCad board)
At the start: 2 copper layers, 18.5 x 46.4 mm, 6 parts, among them U1 MASKROM, U2 29F016/032

Commit message: update img and gerbers
Other:
- board text added: "snes tsop2maskrom rev2 papkor 05.26 vk.com/games_hw"
- board text removed: "snes tsop2maskrom papkor 05.26 rev.2 vk.com/ game_console_hw"
Changed lines of the file:
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@@
 			(plot_on_all_layers_selection 0x00000000_00000000_00000000_00000000)
 			(disableapertmacros no)
-			(usegerberextensions no)
+			(usegerberextensions yes)
 			(usegerberattributes yes)
 			(usegerberadvancedattributes yes)
@@
 			(outputformat 1)
 			(mirror no)
-			(drillshape 1)
+			(drillshape 0)
 			(scaleselection 1)
-			(outputdirectory "")
+			(outputdirectory "gerber")
 		)
 	)
@@
 		(layer "Edge.Cuts")
 	)
-	(gr_text "snes\ntsop2maskrom\npapkor 05.26\nrev.2 vk.com/\ngame_console_hw"
+	(gr_text "snes\ntsop2maskrom rev2\npapkor 05.26\nvk.com/games_hw"
 		(at 121.539 109.347 0)
 		(layer "B.SilkS")
 		(effects
 			(font
-				(size 1 1)
-				(thickness 0.25)
+				(size 1 0.9)
+				(thickness 0.225)
 				(bold yes)
 			)
