File: snes_maskrom_tsop_to_fx_adapter/snes_maskrom_tsop_to_fx_adapter.kicad_pcb (KiCad board)
At the start: 2 copper layers, 27.8 x 16.4 mm, 8 parts, among them U1_1 MASKROM, U1_2 MASKROM, U2 29F016/032

Commit message: update img and gerbers
Other:
- board text added: "papkor 05.26 vk.com/games_hw"
- board text added: "snes tsop2fx rev2"
- board text removed: "papkor 11.25"
- board text removed: "snes tsop2fx rev1.2"
Changed lines of the file:
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@@
 		(layer "Edge.Cuts")
 	)
-	(gr_text "snes tsop2fx rev1.2"
+	(gr_text "snes tsop2fx rev2"
 		(at 38.5826 30.2768 0)
 		(layer "F.SilkS")
@@
 		)
 	)
-	(gr_text "papkor 11.25"
-		(at 45.7454 20.828 90)
+	(gr_text "papkor 05.26\nvk.com/games_hw"
+		(at 45.3644 20.7772 90)
 		(layer "F.SilkS")
 		(effects
 			(font
-				(size 0.5 0.5)
-				(thickness 0.125)
+				(size 0.5 0.4)
+				(thickness 0.1)
 				(bold yes)
 			)
